File: RPi_cape/valve_detect.sch (KiCad schematic (older format))
At the start: 22 parts, among them Q1 MMBT3904, U36 LMC7101B, U37 LMC7101B

Commit message: Manufacturing clean-up
Corrections and additions to BOM etc. for manufacturing
Added power draw tracking spreadsheet
Parts:
- C50: Manufacturer Murata -> AVX; Part Number GRM1885C1H103JA01D -> 06035A102JAT2A
Changed lines of the file:
@@
 F 2 "Capacitor_SMD:C_0603_1608Metric" H 2188 3200 50  0001 C CNN
 F 3 "~" H 2150 3350 50  0001 C CNN
-F 4 "Murata" H 2150 3350 50  0001 C CNN "Manufacturer"
-F 5 "GRM1885C1H103JA01D" H 2150 3350 50  0001 C CNN "Part Number"
+F 4 "AVX" H 2150 3350 50  0001 C CNN "Manufacturer"
+F 5 "06035A102JAT2A" H 2150 3350 50  0001 C CNN "Part Number"
 	1    2150 3350
 	-1   0    0    1
